Commit message: Add files via upload

File: box_urdf/urdf/Box.urdf (robot description, URDF)
Before this commit: robot test_model, 2 links, 1 joints
Links:
- link base_footprint: geometry 
- link base_link: geometry collision cylinder length=0.5 radius=0.25; visual box size=2.0 2.0 0.3
Joints:
- joint base_link_joint: origin xyz=0.0 0 1.25 rpy=0 0 0 -> xyz=2.0 3.0 0.3 rpy=0 0 0
